Commit message: lidar

File: src/car_description/urdf/buggy3.urdf.xacro (robot description, xacro)
@@ -27,4 +27,24 @@
             <geometry>
                 <box size="0.3 0.09 0.16" />
+            </geometry>
+        </collision>
+    </link>
+    <!-- ray -->
+    <link name="MR-Buggy3/GpuLidar">
+        <inertial>
+            <origin xyz="0.0 0.0 0.0" rpy="0.0 0.0 0.0" />
+            <mass value="0.01" />
+            <inertia ixx="0.0001" ixy="0.0" ixz="0.0" iyy="0.0001" iyz="0.0" izz="0.0001" />
+        </inertial>
+        <visual>
+            <origin xyz="0.0 0.0 0.0" rpy="0.0 0.0 0.0" />
+            <geometry>
+                <sphere radius="0.001" />
+            </geometry>
+        </visual>
+        <collision>
+            <origin xyz="0.0 0.0 0.0" rpy="0.0 0.0 0.0" />
+            <geometry>
+                <sphere radius="0.001" />
             </geometry>
         </collision>
@@ -246,4 +266,12 @@
         <dynamics damping="20" friction="10" />
     </joint>
+    <!-- ray -->
+    <joint name="MR-Buggy3/LidarJoint" type="continuous">
+        <origin xyz="0.0 0.0 0.12" rpy="0.0 0.0 0.0" />
+        <parent link="MR-Buggy3/Base" />
+        <child link="MR-Buggy3/GpuLidar" />
+        <axis xyz="0.0 0.0 1" />
+        <limit lower="0.0" upper="0.0" effort="0.0" velocity="0.0" />
+    </joint>
     <!-- ros2_control -->
     <ros2_control name="IgnitionSystem" type="system">
@@ -305,4 +333,9 @@
             <state_interface name="effort" />
         </joint>
+        <joint name="MR-Buggy3/LidarJoint">
+            <state_interface name="position" />
+            <state_interface name="velocity" />
+            <state_interface name="effort" />
+        </joint>
     </ros2_control>
     <gazebo>
@@ -312,4 +345,39 @@
             <parameters>$(find car_description)/config/car.yaml</parameters>
         </plugin>
+        <plugin
+            filename="ignition-gazebo-sensors-system"
+            name="gz::sim::systems::Sensors">
+            <render_engine>ogre2</render_engine>
+        </plugin>
+    </gazebo>
+    <gazebo reference="MR-Buggy3/GpuLidar">
+        <sensor name='gpu_lidar' type='gpu_lidar'>
+            <always_on>true</always_on>
+            <visualize>true</visualize>
+            <topic>lidar</topic>
+            <update_rate>10</update_rate>
+            <gz_frame_id>MR-Buggy3/GpuLidar</gz_frame_id>
+            <ray>
+                <scan>
+                    <horizontal>
+                        <samples>640</samples>
+                        <resolution>1</resolution>
+                        <min_angle>-3.1415926</min_angle>
+                        <max_angle>3.1415926</max_angle>
+                    </horizontal>
+                    <vertical>
+                        <samples>1</samples>
+                        <resolution>0.01</resolution>
+                        <min_angle>0</min_angle>
+                        <max_angle>0</max_angle>
+                    </vertical>
+                </scan>
+                <range>
+                    <min>0.08</min>
+                    <max>10.0</max>
+                    <resolution>0.01</resolution>
+                </range>
+            </ray>
+        </sensor>
     </gazebo>
 </robot>

Commit message: world 反射率

File: src/car_description/urdf/buggy3.urdf.xacro (robot description, xacro)
@@ -268,5 +268,5 @@
     <!-- ray -->
     <joint name="MR-Buggy3/LidarJoint" type="continuous">
-        <origin xyz="0.0 0.0 0.12" rpy="0.0 0.0 0.0" />
+        <origin xyz="0.0 0.0 0.27" rpy="0.0 0.0 0.0" />
         <parent link="MR-Buggy3/Base" />
         <child link="MR-Buggy3/GpuLidar" />
@@ -361,5 +361,5 @@
                 <scan>
                     <horizontal>
-                        <samples>640</samples>
+                        <samples>3600</samples>
                         <resolution>1</resolution>
                         <min_angle>-3.1415926</min_angle>
@@ -375,7 +375,16 @@
                 <range>
                     <min>0.08</min>
-                    <max>10.0</max>
+                    <max>30.0</max>
                     <resolution>0.01</resolution>
                 </range>
+                <noise>
+                    <type>
+                        gaussian
+                    </type>
+                    <mean>0</mean>
+                    <stddev>
+                        0.01
+                    </stddev>
+                </noise>
             </ray>
         </sensor>

Commit message: 关联、提取、拟合

File: src/car_description/urdf/buggy3.urdf.xacro (robot description, xacro)
@@ -227,5 +227,4 @@
         <limit effort="1500" velocity="60.0" />
         <dynamics damping="0.1" friction="0.1" />
-        <mimic joint="MR-Buggy3/RearRightWheelJoint" />
     </joint>
     <!-- 右后轮关节 -->
@@ -255,5 +254,4 @@
         <limit effort="1500" velocity="60.0" />
         <dynamics damping="0.1" friction="0.1" />
-        <mimic joint="MR-Buggy3/RearLeftWheelJoint" />
     </joint>
     <!-- 左后轮关节 -->
@@ -297,9 +295,5 @@
             <state_interface name="effort" />
         </joint>
-        <!-- <joint name="MR-Buggy3/FrontRightWheelJoint">
-            <command_interface name="velocity">
-                <param name="min">-30</param>
-                <param name="max">30</param>
-            </command_interface>
+        <joint name="MR-Buggy3/FrontRightWheelJoint">
             <state_interface name="position" />
             <state_interface name="velocity" />
@@ -307,12 +301,8 @@
         </joint>
         <joint name="MR-Buggy3/FrontLeftWheelJoint">
-            <command_interface name="velocity">
-                <param name="min">-30</param>
-                <param name="max">30</param>
-            </command_interface>
-            <state_interface name="position" />
-            <state_interface name="velocity" />
-            <state_interface name="effort" />
-        </joint> -->
+            <state_interface name="position" />
+            <state_interface name="velocity" />
+            <state_interface name="effort" />
+        </joint>
         <joint name="MR-Buggy3/RearLeftWheelJoint">
             <command_interface name="velocity">
@@ -345,9 +335,9 @@
             <parameters>$(find car_description)/config/car.yaml</parameters>
         </plugin>
-		 <plugin
-			filename="gz-sim-sensors-system"
-			name="gz::sim::systems::Sensors">
-			<render_engine>ogre2</render_engine>
-		</plugin>
+        <plugin
+            filename="gz-sim-sensors-system"
+            name="gz::sim::systems::Sensors">
+            <render_engine>ogre2</render_engine>
+        </plugin>
     </gazebo>
     <gazebo reference="MR-Buggy3/GpuLidar">

Commit message: rviz

File: src/car_description/urdf/buggy3.urdf.xacro (robot description, xacro)
@@ -2,4 +2,5 @@
 <robot xmlns:xacro="http://www.ros.org/wiki/xacro" name="MR-Buggy3">
     <xacro:macro name="iner">
+        <mass value="0.05" />
         <inertia ixx="0.00003331" ixy="0.0" ixz="0.0" iyy="0.0000204" iyz="0.0" izz="0.0000204" />
     </xacro:macro>
@@ -54,5 +55,4 @@
         <inertial>
             <origin xyz="0.0 0.0 0.0" rpy="0.0 0.0 0.0" />
-            <mass value="0.05" />
             <xacro:iner></xacro:iner>
         </inertial>
@@ -104,5 +104,4 @@
         <inertial>
             <origin xyz="0.0 0.0 0.0" rpy="0.0 0.0 0.0" />
-            <mass value="0.05" />
             <xacro:iner></xacro:iner>
         </inertial>
@@ -154,5 +153,4 @@
         <inertial>
             <origin xyz="0.0 0.0 0.0" rpy="0.0 0.0 0.0" />
-            <mass value="0.05" />
             <xacro:iner></xacro:iner>
         </inertial>
@@ -184,5 +182,4 @@
         <inertial>
             <origin xyz="0.0 0.0 0.0" rpy="0.0 0.0 0.0" />
-            <mass value="0.05" />
             <xacro:iner></xacro:iner>
         </inertial>
