Commit message: CR模型

File: src/car_description/urdf/buggy3.urdf.xacro (robot description, xacro)
@@ -1,271 +1,398 @@
 <?xml version="1.0"?>
 <robot xmlns:xacro="http://www.ros.org/wiki/xacro" name="MR-Buggy3">
-    <xacro:macro name="iner">
-        <mass value="0.05" />
-        <inertia ixx="0.00003331" ixy="0.0" ixz="0.0" iyy="0.0000204" iyz="0.0" izz="0.0000204" />
-    </xacro:macro>
+    <material name="red">
+        <color rgba="1 0.1 0.1 1"/>
+    </material>
+    <material name="black">
+        <color rgba="0.1 0.1 0.1 1"/>
+    </material>
+    <material name="gray">
+        <color rgba="0.3 0.3 0.3 1"/>
+    </material>
+    <material name="yellow">
+        <color rgba="1 0.435 0.002 1"/>
+    </material>
+    <material name="green">
+        <color rgba="0.1 1 0.1 1"/>
+    </material>
     <!-- 底座 -->
-    <link name="MR-Buggy3/Base">
-        <inertial>
-            <origin xyz="0.0 0.0 0.0" rpy="0.0 0.0 0.0" />
+    <link name="footbase">
+        <inertial>
+            <origin xyz="0.0 0.0 0.0" rpy="-1.5707 0.0 -1.5707" />
+            <mass value="100.0" />
+            <inertia ixx="20" ixy="0.0" ixz="0.0" iyy="12" iyz="0.0" izz="32" />
+        </inertial>
+        <visual>
+            <origin xyz="0.0 0.0 0.0" rpy="-1.5707 0.0 -1.5707" />
+            <geometry>
+                <mesh filename="package://car_description/meshes/footbase.stl" scale="0.0010 0.0010 0.0010" />
+            </geometry>
+            <material name="black" />
+        </visual>
+        <collision>
+            <origin xyz="0.0 0.0 0.0" rpy="-1.5707 0.0 -1.5707" />
+            <geometry>
+                <mesh filename="package://car_description/meshes/footbase.stl" scale="0.0010 0.0010 0.0010" />
+            </geometry>
+        </collision>
+    </link>
+    <!-- 外壳 -->
+    <link name="out_face">
+        <inertial>
+            <origin xyz="0.0 0.0 0.0" rpy="-1.5707 0.0 -1.5707" />
+            <mass value="100.0" />
+            <inertia ixx="20" ixy="0.0" ixz="0.0" iyy="12" iyz="0.0" izz="12" />
+        </inertial>
+        <visual>
+            <origin xyz="0.0 0.0 0.0" rpy="-1.5707 0.0 -1.5707" />
+            <geometry>
+                <mesh filename="package://car_description/meshes/outface.stl" scale="0.0010 0.0010 0.0010" />
+            </geometry>
+            <material name="yellow" />
+        </visual>
+        <collision>
+            <origin xyz="0.0 0.0 0.0" rpy="-1.5707 0.0 -1.5707" />
+            <geometry>
+                <mesh filename="package://car_description/meshes/outface.stl" scale="0.0010 0.0010 0.0010" />
+            </geometry>
+        </collision>
+    </link>
+    <!-- 叉齿架 -->
+    <link name="fork_frame">
+        <inertial>
+            <origin xyz="0.0 0.0 0.0" rpy="-1.5707 0.0 -1.5707" />
+            <mass value="200.0" />
+            <inertia ixx="40" ixy="0.0" ixz="0.0" iyy="12" iyz="0.0" izz="12" />
+        </inertial>
+        <visual>
+            <origin xyz="0 0.0 0.00" rpy="-1.5707 0.0 -1.5707" />
+            <geometry>
+                <mesh filename="package://car_description/meshes/frame.stl" scale="0.0010 0.0010 0.0010" />
+            </geometry>
+            <material name="black" />
+        </visual>
+        <collision>
+            <origin xyz="0.0 0.0 0.0" rpy="-1.5707 0.0 -1.5707" />
+            <geometry>
+                <mesh filename="package://car_description/meshes/frame.stl" scale="0.0010 0.0010 0.0010" />
+            </geometry>
+        </collision>
+    </link>
+    <!-- 叉齿 -->
+    <link name="fork">
+        <inertial>
+            <origin xyz="0.0 0.0 0.0" rpy="-1.5707 0.0 -1.5707" />
+            <mass value="100.0" />
+            <inertia ixx="50" ixy="0.0" ixz="0.0" iyy="22" iyz="0.0" izz="42" />
+        </inertial>
+        <visual>
+            <origin xyz="0.0 0.0 0.0" rpy="-1.5707 0.0 -1.5707" />
+            <geometry>
+                <mesh filename="package://car_description/meshes/fork.stl" scale="0.0010 0.0010 0.0010" />
+            </geometry>
+            <material name="gray" />
+        </visual>
+        <collision>
+            <origin xyz="0.0 0.0 0.0" rpy="-1.5707 0.0 -1.5707" />
+            <geometry>
+                <mesh filename="package://car_description/meshes/fork.stl" scale="0.0010 0.0010 0.0010" />
+            </geometry>
+        </collision>
+    </link>
+    <!-- 仿撞条 -->
+    <link name="bar">
+        <inertial>
+            <origin xyz="0.0 0.0 0.0" rpy="-1.5707 0.0 -1.5707" />
+            <mass value="20.0" />
+            <inertia ixx="7" ixy="0.0" ixz="0.0" iyy="3" iyz="0.0" izz="5" />
+        </inertial>
+        <visual>
+            <origin xyz="0.0 0.0 0.0" rpy="-1.5707 0.0 -1.5707" />
+            <geometry>
+                <mesh filename="package://car_description/meshes/bar.stl" scale="0.0010 0.0010 0.0010" />
+            </geometry>
+            <material name="black" />
+        </visual>
+        <collision>
+            <origin xyz="0.0 0.0 0.0" rpy="-1.5707 0.0 -1.5707" />
+            <geometry>
+                <mesh filename="package://car_description/meshes/bar.stl" scale="0.0010 0.0010 0.0010" />
+            </geometry>
+        </collision>
+    </link>
+    <!-- 避障雷达 -->
+    <link name="avoid_lidar">
+        <inertial>
+            <origin xyz="0.0 0.0 0.0" rpy="-1.5707 0.0 -1.5707" />
+            <mass value="20.0" />
+            <inertia ixx="7" ixy="0.0" ixz="0.0" iyy="3" iyz="0.0" izz="5" />
+        </inertial>
+        <visual>
+            <origin xyz="0.0 0.0 0.0" rpy="-1.5707 0.0 -1.5707" />
+            <geometry>
+                <mesh filename="package://car_description/meshes/lidar.stl" scale="0.0010 0.0010 0.0010" />
+            </geometry>
+            <material name="green" />
+        </visual>
+        <collision>
+            <origin xyz="0.0 0.0 0.0" rpy="-1.5707 0.0 -1.5707" />
+            <geometry>
+                <mesh filename="package://car_description/meshes/lidar.stl" scale="0.0010 0.0010 0.0010" />
+            </geometry>
+        </collision>
+    </link>
+    <!-- 屏幕 -->
+    <link name="screen">
+        <inertial>
+            <origin xyz="0.0 0.0 0.0" rpy="-1.5707 0.0 -1.5707" />
+            <mass value="5.0" />
+            <inertia ixx="0.7" ixy="0.0" ixz="0.0" iyy="0.3" iyz="0.0" izz="0.5" />
+        </inertial>
+        <visual>
+            <origin xyz="0.0 0.0 0.0" rpy="-1.5707 0.0 -1.5707" />
+            <geometry>
+                <mesh filename="package://car_description/meshes/screen.stl" scale="0.0010 0.0010 0.0010" />
+            </geometry>
+            <material name="black" />
+        </visual>
+        <collision>
+            <origin xyz="0.0 0.0 0.0" rpy="-1.5707 0.0 -1.5707" />
+            <geometry>
+                <mesh filename="package://car_description/meshes/screen.stl" scale="0.0010 0.0010 0.0010" />
+            </geometry>
+        </collision>
+    </link>
+    <!-- 按钮 -->
+    <link name="button">
+        <inertial>
+            <origin xyz="0.0 0.0 0.0" rpy="-1.5707 0.0 -1.5707" />
+            <mass value="5.0" />
+            <inertia ixx="0.7" ixy="0.0" ixz="0.0" iyy="0.3" iyz="0.0" izz="0.5" />
+        </inertial>
+        <visual>
+            <origin xyz="0.0 0.0 0.0" rpy="-1.5707 0.0 -1.5707" />
+            <geometry>
+                <mesh filename="package://car_description/meshes/button.stl" scale="0.0010 0.0010 0.0010" />
+            </geometry>
+            <material name="red" />
+        </visual>
+        <collision>
+            <origin xyz="0.0 0.0 0.0" rpy="-1.5707 0.0 -1.5707" />
+            <geometry>
+                <mesh filename="package://car_description/meshes/button.stl" scale="0.0010 0.0010 0.0010" />
+            </geometry>
+        </collision>
+    </link>
+    <!-- 充电口 -->
+    <link name="charge">
+        <inertial>
+            <origin xyz="0.0 0.0 0.0" rpy="-1.5707 0.0 -1.5707" />
+            <mass value="5.0" />
+            <inertia ixx="0.7" ixy="0.0" ixz="0.0" iyy="0.3" iyz="0.0" izz="0.5" />
+        </inertial>
+        <visual>
+            <origin xyz="0.0 0.0 0.0" rpy="-1.5707 0.0 -1.5707" />
+            <geometry>
+                <mesh filename="package://car_description/meshes/charge.stl" scale="0.0010 0.0010 0.0010" />
+            </geometry>
+            <material name="green" />
+        </visual>
+        <collision>
+            <origin xyz="0.0 0.0 0.0" rpy="-1.5707 0.0 -1.5707" />
+            <geometry>
+                <mesh filename="package://car_description/meshes/charge.stl" scale="0.0010 0.0010 0.0010" />
+            </geometry>
+        </collision>
+    </link>
+    <!-- 光通信口 -->
+    <link name="sun">
+        <inertial>
+            <origin xyz="0.0 0.0 0.0" rpy="-1.5707 0.0 -1.5707" />
+            <mass value="5.0" />
+            <inertia ixx="0.7" ixy="0.0" ixz="0.0" iyy="0.3" iyz="0.0" izz="0.5" />
+        </inertial>
+        <visual>
+            <origin xyz="0.0 0.0 0.0" rpy="-1.5707 0.0 -1.5707" />
+            <geometry>
+                <mesh filename="package://car_description/meshes/sun.stl" scale="0.0010 0.0010 0.0010" />
+            </geometry>
+            <material name="green" />
+        </visual>
+        <collision>
+            <origin xyz="0.0 0.0 0.0" rpy="-1.5707 0.0 -1.5707" />
+            <geometry>
+                <mesh filename="package://car_description/meshes/sun.stl" scale="0.0010 0.0010 0.0010" />
+            </geometry>
+        </collision>
+    </link>
+    <!-- 主舵轮 -->
+    <link name="main_wheel_link">
+        <inertial>
+            <origin xyz="0 0.0 0.0" rpy="-1.5707 0.0 0" />
+            <mass value="100.0" />
+            <inertia ixx="50" ixy="0.0" ixz="0.0" iyy="42" iyz="0.0" izz="22" />
+        </inertial>
+        <visual>
+            <origin xyz="0 0.0 0.0" rpy="-1.5707 0.0 0" />
+            <geometry>
+                <cylinder radius="0.105" length="0.075"/>
+            </geometry>
+            <material name="gray"/>
+        </visual>
+        <visual>
+            <origin xyz="0 0.0 0.00" rpy="-1.5707 0.0 0" />
+            <geometry>
+                <cylinder radius="0.105" length="0.075"/>
+            </geometry>
+        </visual>
+        <collision>
+            <origin xyz="0 0.0 0.0" rpy="-1.5707 0.0 0" />
+            <geometry>
+                <cylinder radius="0.105" length="0.075"/>
+            </geometry>
+        </collision>
+    </link>
+    <!-- 左前轮 -->
+    <link name="left_wheel_link">
+        <inertial>
+            <origin xyz="0 0.0 0.0" rpy="0 0.0 0" />
+            <mass value="30.0" />
+            <inertia ixx="10" ixy="0.0" ixz="0.0" iyy="12" iyz="0.0" izz="12" />
+        </inertial>
+        <visual>
+            <origin xyz="0 0.0 0.0" rpy="0 0.0 0" />
+            <geometry>
+                <mesh filename="package://car_description/meshes/frontwheel.stl" scale="0.0010 0.0010 0.0010" />
+            </geometry>
+            <material name="gray"/>
+        </visual>
+        <collision>
+            <origin xyz="0 0.0 0.0" rpy="0 0.0 0" />
+            <geometry>
+                <mesh filename="package://car_description/meshes/frontwheel.stl" scale="0.0010 0.0010 0.0010" />
+            </geometry>
+        </collision>
+    </link>
+    <!-- 右前轮 -->
+    <link name="right_wheel_link">
+        <inertial>
+            <origin xyz="0 0.0 0.0" rpy="0 0.0 0" />
+            <mass value="30.0" />
+            <inertia ixx="10" ixy="0.0" ixz="0.0" iyy="12" iyz="0.0" izz="12" />
+        </inertial>
+        <visual>
+            <origin xyz="0 0.0 0.0" rpy="0 0.0 0" />
+            <geometry>
+                <mesh filename="package://car_description/meshes/frontwheel.stl" scale="0.0010 0.0010 0.0010" />
+            </geometry>
+            <material name="gray"/>
+        </visual>
+        <collision>
+            <origin xyz="0 0.0 0.0" rpy="0 0.0 0" />
+            <geometry>
+                <mesh filename="package://car_description/meshes/frontwheel.stl" scale="0.0010 0.0010 0.0010" />
+            </geometry>
+        </collision>
+    </link>
+    <!-- 主轮转向轴 -->
+    <link name="main_wheel_base_link">
+        <inertial>
+            <origin xyz="0 0.0 0.0" rpy="0 0.0 0" />
+            <mass value="100.0" />
+            <inertia ixx="20" ixy="0.0" ixz="0.0" iyy="12" iyz="0.0" izz="12" />
+        </inertial>
+    </link>
+    <!-- 导航2D雷达 -->
+    <link name="main_2d_lidar_link">
+        <inertial>
+            <origin xyz="0 0.0 0.0" rpy="0 0.0 0" />
             <mass value="3.0" />
-            <inertia ixx="0.054" ixy="0.0" ixz="0.0" iyy="0.252" iyz="0.0" izz="0.252" />
-        </inertial>
-        <visual>
-            <origin xyz="0.1371 0.0 -0.0115" rpy="-0.018 0.0 1.5707" />
-            <geometry>
-                <mesh filename="package://car_description/meshes/BaseReduced.dae" />
-            </geometry>
-        </visual>
-        <visual>
-            <origin xyz="0.1371 0.0 -0.0115" rpy="-0.018 0.0 1.5707" />
-            <geometry>
-                <mesh filename="package://car_description/meshes/TopReduced.dae" />
-            </geometry>
-        </visual>
-        <collision>
-            <origin xyz="0.0 0.0 0.09" rpy="0.0 0.0 0.0" />
-            <geometry>
-                <box size="0.3 0.09 0.16" />
-            </geometry>
-        </collision>
-    </link>
-    <!-- ray -->
-    <link name="MR-Buggy3/GpuLidar">
-        <inertial>
-            <origin xyz="0.0 0.0 0.0" rpy="0.0 0.0 0.0" />
-            <mass value="0.01" />
-            <inertia ixx="0.0001" ixy="0.0" ixz="0.0" iyy="0.0001" iyz="0.0" izz="0.0001" />
-        </inertial>
-        <visual>
-            <origin xyz="0.0 0.0 0.0" rpy="0.0 0.0 0.0" />
-            <geometry>
-                <sphere radius="0.001" />
-            </geometry>
-        </visual>
-        <collision>
-            <origin xyz="0.0 0.0 0.0" rpy="0.0 0.0 0.0" />
-            <geometry>
-                <sphere radius="0.001" />
-            </geometry>
-        </collision>
-    </link>
-    <!-- 右前轮 -->
-    <link name="MR-Buggy3/FrontRightWheel">
-        <inertial>
-            <origin xyz="0.0 0.0 0.0" rpy="0.0 0.0 0.0" />
-            <xacro:iner></xacro:iner>
-        </inertial>
-        <visual name="">
-            <origin xyz="0.0 -0.01 0.0" rpy="0.0 0.0 0.0" />
-            <geometry>
-                <mesh filename="package://car_description/meshes/Wheel.dae" />
-            </geometry>
-        </visual>
-        <collision>
-            <origin xyz="0.0 0.012 0.0" rpy="1.5707 0.0 0.0" />
-            <geometry>
-                <cylinder radius="0.0365" length="0.03" />
-            </geometry>
-            <surface>
-                <friction>
-                    <ode>
-                        <mu>1</mu>
-                        <mu2>1</mu2>
-                        <slip1>1.0</slip1>
-                        <slip2>1.0</slip2>
-                    </ode>
-                </friction>
-            </surface>
-        </collision>
-    </link>
-    <!-- 右前轮转向 -->
-    <link name="MR-Buggy3/FrontRightWheelSteering">
-        <visual>
-            <origin xyz="0.0 0.0 0.0" rpy="0.0 0.0 0.0" />
-            <geometry>
-                <sphere radius="0.001" />
-            </geometry>
-        </visual>
-        <collision>
-            <origin xyz="0.0 0.0 0.0" rpy="0.0 0.0 0.0" />
-            <geometry>
-                <sphere radius="0.001" />
-            </geometry>
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
Commit message: CR can driver

File: src/car_description/urdf/buggy3.urdf.xacro (robot description, xacro)
@@ -41,6 +41,6 @@
         <inertial>
             <origin xyz="0.0 0.0 0.0" rpy="-1.5707 0.0 -1.5707" />
-            <mass value="100.0" />
-            <inertia ixx="20" ixy="0.0" ixz="0.0" iyy="12" iyz="0.0" izz="12" />
+            <mass value="300.0" />
+            <inertia ixx="48" ixy="0.0" ixz="0.0" iyy="58" iyz="0.0" izz="22" />
         </inertial>
         <visual>
@@ -83,6 +83,6 @@
         <inertial>
             <origin xyz="0.0 0.0 0.0" rpy="-1.5707 0.0 -1.5707" />
-            <mass value="100.0" />
-            <inertia ixx="50" ixy="0.0" ixz="0.0" iyy="22" iyz="0.0" izz="42" />
+            <mass value="46.0" />
+            <inertia ixx="0.09" ixy="0.0" ixz="0.0" iyy="0.97" iyz="0.0" izz="1" />
         </inertial>
         <visual>
@@ -230,6 +230,6 @@
         <inertial>
             <origin xyz="0 0.0 0.0" rpy="-1.5707 0.0 0" />
-            <mass value="100.0" />
-            <inertia ixx="50" ixy="0.0" ixz="0.0" iyy="42" iyz="0.0" izz="22" />
+            <mass value="6.79" />
+            <inertia ixx="0.089" ixy="0.0" ixz="0.0" iyy="0.089" iyz="0.0" izz="0.172" />
         </inertial>
         <visual>
@@ -298,7 +298,15 @@
     <link name="main_wheel_base_link">
         <inertial>
-            <origin xyz="0 0.0 0.0" rpy="0 0.0 0" />
-            <mass value="100.0" />
-            <inertia ixx="20" ixy="0.0" ixz="0.0" iyy="12" iyz="0.0" izz="12" />
+            <origin xyz="0.0 0.0 0.0" rpy="0.0 0.0 0.0" />
+            <mass value="3.0" />
+            <inertia ixx="0.054" ixy="0.0" ixz="0.0" iyy="0.252" iyz="0.0" izz="0.252" />
+        </inertial>
+    </link>
+    <!-- base_link -->
+    <link name="base_link">
+        <inertial>
+            <origin xyz="0.0 0.0 0.0" rpy="0.0 0.0 0.0" />
+            <mass value="3.0" />
+            <inertia ixx="0.054" ixy="0.0" ixz="0.0" iyy="0.252" iyz="0.0" izz="0.252" />
         </inertial>
     </link>
@@ -361,14 +369,14 @@
         <child link="fork"/>
         <axis xyz="0.0 0.0 1"/>
-        <limit lower="0" upper="3.0" effort="20.0" velocity="2.0"/>
-        <dynamics damping="1.0" friction="0.5"/>
-    </joint>
-    <joint name="main_wheel_base_joint" type="revolute">
+        <limit lower="-1" upper="3.0" effort="3000.0" velocity="1.0"/>
+        <dynamics damping="100.0" friction="10"/>
+    </joint>
+    <joint name="main_wheel_base_joint" type="continuous">
         <origin xyz="0.21 0.0 0.04" rpy="0.0 0.0 0.0"/>
         <parent link="footbase"/>
         <child link="main_wheel_base_link"/>
         <axis xyz="0.0 0.0 1"/>
-        <limit lower="-1.5707" upper="1.5707" effort="20.0" velocity="1.5707"/>
-        <dynamics damping="1.0" friction="0.5"/>
+        <limit effort="500.0" velocity="1"/>
+        <dynamics damping="1.0" friction="1"/>
     </joint>
     <joint name="main_wheel_joint" type="continuous">
@@ -377,6 +385,6 @@
         <child link="main_wheel_link"/>
         <axis xyz="0.0 1.0 0.0"/>
-        <limit lower="-100" upper="100.0" effort="20.0" velocity="2.0"/>
-        <dynamics damping="1.0" friction="0.5"/>
+        <limit effort="1600.0" velocity="20.0"/>
+        <dynamics damping="4.0" friction="1.5"/>
     </joint>
     <joint name="left_wheel_joint" type="continuous">
@@ -395,4 +403,10 @@
         <limit lower="-100" upper="100.0" effort="20.0" velocity="2.0"/>
         <dynamics damping="1.0" friction="0.5"/>
+    </joint>
+    <joint name="base_link_joint" type="fixed">
+        <origin xyz="-1.01 0 0" rpy="0.0 0.0 0"/>
+        <parent link="footbase"/>
+        <child link="base_link"/>
+        <axis xyz="0.0 0.0 0.0"/>
     </joint>
     <!-- ros2_control -->
@@ -424,4 +438,14 @@
                 <param name="max">30</param>
             </command_interface>
+            <state_interface name="position" />
+            <state_interface name="velocity" />
+            <state_interface name="effort" />
+        </joint>
+        <joint name="left_wheel_joint">
+            <state_interface name="position" />
+            <state_interface name="velocity" />
+            <state_interface name="effort" />
+        </joint>
+        <joint name="right_wheel_joint">
             <state_interface name="position" />
             <state_interface name="velocity" />

Commit message: 修复物理参数打滑问题

File: src/car_description/urdf/buggy3.urdf.xacro (robot description, xacro)
@@ -251,4 +251,15 @@
                 <cylinder radius="0.105" length="0.075"/>
             </geometry>
+            <surface>
+                <friction>
+                    <ode>
+                        <mu>1.0</mu>
+                        <mu2>100</mu2>
+                        <fdir1>0 0 0</fdir1>
+                        <slip1>0.02</slip1>
+                        <slip2>0</slip2>
+                    </ode>
+                </friction>
+            </surface>
         </collision>
     </link>
@@ -272,4 +283,15 @@
                 <mesh filename="package://car_description/meshes/frontwheel.stl" scale="0.0010 0.0010 0.0010" />
             </geometry>
+            <surface>
+                <friction>
+                    <ode>
+                        <mu>1.0</mu>
+                        <mu2>100</mu2>
+                        <fdir1>0 0 0</fdir1>
+                        <slip1>0.02</slip1>
+                        <slip2>0</slip2>
+                    </ode>
+                </friction>
+            </surface>
         </collision>
     </link>
@@ -293,4 +315,15 @@
                 <mesh filename="package://car_description/meshes/frontwheel.stl" scale="0.0010 0.0010 0.0010" />
             </geometry>
+            <surface>
+                <friction>
+                    <ode>
+                        <mu>1.0</mu>
+                        <mu2>100</mu2>
+                        <fdir1>0 0 0</fdir1>
+                        <slip1>0.02</slip1>
+                        <slip2>0</slip2>
+                    </ode>
+                </friction>
+            </surface>
         </collision>
     </link>
@@ -386,5 +419,5 @@
         <axis xyz="0.0 1.0 0.0"/>
         <limit effort="1600.0" velocity="20.0"/>
-        <dynamics damping="4.0" friction="1.5"/>
+        <dynamics damping="4.0" friction="10.0" friction2="100.0"/>
     </joint>
     <joint name="left_wheel_joint" type="continuous">
@@ -394,5 +427,5 @@
         <axis xyz="1.0 0.0 0.0"/>
         <limit lower="-100" upper="100.0" effort="20.0" velocity="2.0"/>
-        <dynamics damping="1.0" friction="0.5"/>
+        <dynamics damping="1.0" friction="10.0" friction2="100.0"/>
     </joint>
     <joint name="right_wheel_joint" type="continuous">
@@ -402,5 +435,5 @@
         <axis xyz="1.0 0.0 0.0"/>
         <limit lower="-100" upper="100.0" effort="20.0" velocity="2.0"/>
-        <dynamics damping="1.0" friction="0.5"/>
+        <dynamics damping="1.0" friction="10.0" friction2="100.0"/>
     </joint>
     <joint name="base_link_joint" type="fixed">
@@ -484,5 +517,5 @@
                 <range>
                     <min>0.08</min>
-                    <max>10.0</max>
+                    <max>50.0</max>
                     <resolution>0.01</resolution>
                 </range>
