Commit message: odom

File: src/car_description/urdf/buggy3.urdf.xacro (robot description, xacro)
@@ -1,4 +1,4 @@
 <?xml version="1.0"?>
-<robot xmlns:xacro="http://www.ros.org/wiki/xacro" name="MR-Buggy3">
+<robot xmlns:xacro="http://www.ros.org/wiki/xacro" name="ZC_CR">
     <material name="red">
         <color rgba="1 0.1 0.1 1"/>
@@ -18,8 +18,13 @@
     <!-- 底座 -->
     <link name="footbase">
-        <inertial>
-            <origin xyz="0.0 0.0 0.0" rpy="-1.5707 0.0 -1.5707" />
+        <!-- <inertial>
+            <origin xyz="0.0 0.0 0.4" rpy="-1.5707 0.0 -1.5707" />
             <mass value="100.0" />
-            <inertia ixx="20" ixy="0.0" ixz="0.0" iyy="12" iyz="0.0" izz="32" />
+            <inertia ixx="2.167" ixy="0.0" ixz="0.0" iyy="12.083" iyz="0.0" izz="14.083" />
+        </inertial> -->
+        <inertial auto="true">
+            <mass value="100.0" />
+            <origin xyz="0.0 0.0 0.4" rpy="-1.5707 0.0 -1.5707" />
+            <inertia ixx="2.167" ixy="0.0" ixz="0.0" iyy="12.083" iyz="0.0" izz="20" />
         </inertial>
         <visual>
@@ -31,4 +36,5 @@
         </visual>
         <collision>
+            <density>7874</density>
             <origin xyz="0.0 0.0 0.0" rpy="-1.5707 0.0 -1.5707" />
             <geometry>
@@ -39,8 +45,13 @@
     <!-- 外壳 -->
     <link name="out_face">
-        <inertial>
-            <origin xyz="0.0 0.0 0.0" rpy="-1.5707 0.0 -1.5707" />
-            <mass value="300.0" />
-            <inertia ixx="48" ixy="0.0" ixz="0.0" iyy="58" iyz="0.0" izz="22" />
+        <!-- <inertial>
+            <origin xyz="0.0 0.0 0.0" rpy="-1.5707 0.0 -1.5707" />
+            <mass value="20.0" />
+            <inertia ixx="1.933" ixy="0.0" ixz="0.0" iyy="2.733" iyz="0.0" izz="1.333" />
+        </inertial> -->
+        <inertial auto="true">
+            <origin xyz="0.0 0.0 0.0" rpy="-1.5707 0.0 -1.5707" />
+            <mass value="20.0" />
+            <inertia ixx="1.933" ixy="0.0" ixz="0.0" iyy="2.733" iyz="0.0" izz="1.333" />
         </inertial>
         <visual>
@@ -52,4 +63,5 @@
         </visual>
         <collision>
+            <density>7874</density>
             <origin xyz="0.0 0.0 0.0" rpy="-1.5707 0.0 -1.5707" />
             <geometry>
@@ -60,8 +72,13 @@
     <!-- 叉齿架 -->
     <link name="fork_frame">
-        <inertial>
-            <origin xyz="0.0 0.0 0.0" rpy="-1.5707 0.0 -1.5707" />
-            <mass value="200.0" />
-            <inertia ixx="40" ixy="0.0" ixz="0.0" iyy="12" iyz="0.0" izz="12" />
+        <!-- <inertial>
+            <origin xyz="0.0 0.0 0.0" rpy="-1.5707 0.0 -1.5707" />
+            <mass value="80.0" />
+            <inertia ixx="28.83" ixy="0.0" ixz="0.0" iyy="26.83" iyz="0.0" izz="1.333" />
+        </inertial> -->
+        <inertial auto="true">
+            <origin xyz="0.0 0.0 0.0" rpy="-1.5707 0.0 -1.5707" />
+            <mass value="80.0" />
+            <inertia ixx="28.83" ixy="0.0" ixz="0.0" iyy="26.83" iyz="0.0" izz="1.333" />
         </inertial>
         <visual>
@@ -73,4 +90,5 @@
         </visual>
         <collision>
+            <density>7874</density>
             <origin xyz="0.0 0.0 0.0" rpy="-1.5707 0.0 -1.5707" />
             <geometry>
@@ -81,8 +99,13 @@
     <!-- 叉齿 -->
     <link name="fork">
-        <inertial>
-            <origin xyz="0.0 0.0 0.0" rpy="-1.5707 0.0 -1.5707" />
+        <!-- <inertial>
+            <origin xyz="-0.9 0.0 0.0" rpy="-1.5707 0.0 -1.5707" />
             <mass value="46.0" />
             <inertia ixx="0.09" ixy="0.0" ixz="0.0" iyy="0.97" iyz="0.0" izz="1" />
+        </inertial> -->
+        <inertial auto="true">
+            <origin xyz="-0.9 0.0 0.0" rpy="-1.5707 0.0 -1.5707" />
+            <mass value="30.0" />
+            <inertia ixx="0.09" ixy="0.0" ixz="0.0" iyy="0.97" iyz="0.0" izz="1" />
         </inertial>
         <visual>
@@ -94,4 +117,5 @@
         </visual>
         <collision>
+            <density>7874</density>
             <origin xyz="0.0 0.0 0.0" rpy="-1.5707 0.0 -1.5707" />
             <geometry>
@@ -102,8 +126,13 @@
     <!-- 仿撞条 -->
     <link name="bar">
-        <inertial>
-            <origin xyz="0.0 0.0 0.0" rpy="-1.5707 0.0 -1.5707" />
-            <mass value="20.0" />
-            <inertia ixx="7" ixy="0.0" ixz="0.0" iyy="3" iyz="0.0" izz="5" />
+        <!-- <inertial>
+            <origin xyz="0.0 0.0 0.0" rpy="-1.5707 0.0 -1.5707" />
+            <mass value="1.0" />
+            <inertia ixx="0.01" ixy="0.0" ixz="0.0" iyy="0.01" iyz="0.0" izz="0.0042" />
+        </inertial> -->
+        <inertial auto="true">
+            <origin xyz="0.0 0.0 0.0" rpy="-1.5707 0.0 -1.5707" />
+            <mass value="1.0" />
+            <inertia ixx="0.01" ixy="0.0" ixz="0.0" iyy="0.01" iyz="0.0" izz="0.0042" />
         </inertial>
         <visual>
@@ -115,4 +144,5 @@
         </visual>
         <collision>
+            <density>800</density>
             <origin xyz="0.0 0.0 0.0" rpy="-1.5707 0.0 -1.5707" />
             <geometry>
@@ -123,8 +153,13 @@
     <!-- 避障雷达 -->
     <link name="avoid_lidar">
-        <inertial>
-            <origin xyz="0.0 0.0 0.0" rpy="-1.5707 0.0 -1.5707" />
-            <mass value="20.0" />
-            <inertia ixx="7" ixy="0.0" ixz="0.0" iyy="3" iyz="0.0" izz="5" />
+        <!-- <inertial>
+            <origin xyz="0.0 0.0 0.0" rpy="-1.5707 0.0 -1.5707" />
+            <mass value="2.0" />
+            <inertia ixx="0.01" ixy="0.0" ixz="0.0" iyy="0.01" iyz="0.0" izz="0.0042"/>
+        </inertial> -->
+        <inertial auto="true">
+            <origin xyz="0.0 0.0 0.0" rpy="-1.5707 0.0 -1.5707" />
+            <mass value="1.0" />
+            <inertia ixx="0.01" ixy="0.0" ixz="0.0" iyy="0.01" iyz="0.0" izz="0.0042"/>
         </inertial>
         <visual>
@@ -136,4 +171,5 @@
         </visual>
         <collision>
+            <density>1800</density>
             <origin xyz="0.0 0.0 0.0" rpy="-1.5707 0.0 -1.5707" />
             <geometry>
@@ -144,8 +180,13 @@
     <!-- 屏幕 -->
     <link name="screen">
-        <inertial>
+        <!-- <inertial>
             <origin xyz="0.0 0.0 0.0" rpy="-1.5707 0.0 -1.5707" />
             <mass value="5.0" />
             <inertia ixx="0.7" ixy="0.0" ixz="0.0" iyy="0.3" iyz="0.0" izz="0.5" />
+        </inertial> -->
+        <inertial auto="true">
+            <origin xyz="0.0 0.0 0.0" rpy="-1.5707 0.0 -1.5707" />
+            <mass value="1.0" />
+            <inertia ixx="0.7" ixy="0.0" ixz="0.0" iyy="0.3" iyz="0.0" izz="0.5" />
         </inertial>
         <visual>
@@ -157,4 +198,5 @@
         </visual>
         <collision>
+            <density>1100</density>
             <origin xyz="0.0 0.0 0.0" rpy="-1.5707 0.0 -1.5707" />
             <geometry>
@@ -165,8 +207,13 @@
     <!-- 按钮 -->
     <link name="button">
-        <inertial>
+        <!-- <inertial>
             <origin xyz="0.0 0.0 0.0" rpy="-1.5707 0.0 -1.5707" />
             <mass value="5.0" />
             <inertia ixx="0.7" ixy="0.0" ixz="0.0" iyy="0.3" iyz="0.0" izz="0.5" />
+        </inertial> -->
+        <inertial auto="true">
+            <origin xyz="0.0 0.0 0.0" rpy="-1.5707 0.0 -1.5707" />
+            <mass value="0.1" />
+            <inertia ixx="0.7" ixy="0.0" ixz="0.0" iyy="0.3" iyz="0.0" izz="0.5" />
         </inertial>
         <visual>
@@ -178,4 +225,5 @@
         </visual>
         <collision>
+            <density>400</density>
             <origin xyz="0.0 0.0 0.0" rpy="-1.5707 0.0 -1.5707" />
             <geometry>
@@ -186,8 +234,13 @@
     <!-- 充电口 -->
     <link name="charge">
-        <inertial>
+        <!-- <inertial>
             <origin xyz="0.0 0.0 0.0" rpy="-1.5707 0.0 -1.5707" />
             <mass value="5.0" />
             <inertia ixx="0.7" ixy="0.0" ixz="0.0" iyy="0.3" iyz="0.0" izz="0.5" />
+        </inertial> -->
+        <inertial auto="true">
+            <origin xyz="0.0 0.0 0.0" rpy="-1.5707 0.0 -1.5707" />
+            <mass value="1.0" />
+            <inertia ixx="0.7" ixy="0.0" ixz="0.0" iyy="0.3" iyz="0.0" izz="0.5" />
         </inertial>
         <visual>
@@ -199,4 +252,5 @@
         </visual>
         <collision>
+            <density>7874</density>
             <origin xyz="0.0 0.0 0.0" rpy="-1.5707 0.0 -1.5707" />
             <geometry>
@@ -207,8 +261,13 @@
     <!-- 光通信口 -->
     <link name="sun">
-        <inertial>
+        <!-- <inertial>
             <origin xyz="0.0 0.0 0.0" rpy="-1.5707 0.0 -1.5707" />
             <mass value="5.0" />
             <inertia ixx="0.7" ixy="0.0" ixz="0.0" iyy="0.3" iyz="0.0" izz="0.5" />
+        </inertial> -->
+        <inertial auto="true">
+            <origin xyz="0.0 0.0 0.0" rpy="-1.5707 0.0 -1.5707" />
+            <mass value="1.0" />
+            <inertia ixx="0.7" ixy="0.0" ixz="0.0" iyy="0.3" iyz="0.0" izz="0.5" />
         </inertial>
         <visual>
@@ -220,4 +279,5 @@
         </visual>
         <collision>
+            <density>7874</density>
             <origin xyz="0.0 0.0 0.0" rpy="-1.5707 0.0 -1.5707" />
             <geometry>
@@ -228,11 +288,16 @@
     <!-- 主舵轮 -->
     <link name="main_wheel_link">
-        <inertial>
+        <!-- <inertial>
             <origin xyz="0 0.0 0.0" rpy="-1.5707 0.0 0" />
             <mass value="6.79" />
-            <inertia ixx="0.089" ixy="0.0" ixz="0.0" iyy="0.089" iyz="0.0" izz="0.172" />
-        </inertial>
-        <visual>
+            <inertia ixx="0.244" ixy="0.0" ixz="0.0" iyy="0.244" iyz="0.0" izz="0.172" />
+        </inertial> -->
+        <inertial auto="true">
             <origin xyz="0 0.0 0.0" rpy="-1.5707 0.0 0" />
+            <mass value="20.0" />
+            <inertia ixx="0.244" ixy="0.0" ixz="0.0" iyy="0.244" iyz="0.0" izz="0.172" />
+        </inertial>
+        <visual>
+            <origin xyz="0 0.0 0.0" rpy="-1.5707 0.0 0" />
             <geometry>
                 <cylinder radius="0.105" length="0.075"/>
@@ -247,4 +312,5 @@
         </visual>
         <collision>
+            <density>4000</density>
             <origin xyz="0 0.0 0.0" rpy="-1.5707 0.0 0" />
             <geometry>
@@ -254,9 +320,6 @@
                 <friction>
                     <ode>
-                        <mu>1.0</mu>
-                        <mu2>100</mu2>
-                        <fdir1>0 0 0</fdir1>
-                        <slip1>0.02</slip1>
-                        <slip2>0</slip2>
+                        <mu>10000000</mu>
+                        <mu2>10000000</mu2>
                     </ode>
                 </friction>
@@ -266,11 +329,16 @@
     <!-- 左前轮 -->
     <link name="left_wheel_link">
-        <inertial>
+        <!-- <inertial>
+            <origin xyz="0 0.0 0.0" rpy="-1.5707 0.0 -1.5707" />
+            <mass value="30.0" />
+            <inertia ixx="0.089" ixy="0.0" ixz="0.0" iyy="0.089" iyz="0.0" izz="0.172" />
+        </inertial> -->
+        <inertial auto="true">
+            <origin xyz="0 0.0 0.0" rpy="-1.5707 0.0 -1.5707" />
+            <mass value="5.0" />
+            <inertia ixx="0.089" ixy="0.0" ixz="0.0" iyy="0.089" iyz="0.0" izz="0.172" />
+        </inertial>
+        <visual>
             <origin xyz="0 0.0 0.0" rpy="0 0.0 0" />
-            <mass value="30.0" />
-            <inertia ixx="10" ixy="0.0" ixz="0.0" iyy="12" iyz="0.0" izz="12" />
-        </inertial>
-        <visual>
-            <origin xyz="0 0.0 0.0" rpy="0 0.0 0" />
             <geometry>
                 <mesh filename="package://car_description/meshes/frontwheel.stl" scale="0.0010 0.0010 0.0010" />
@@ -279,4 +347,5 @@
         </visual>
         <collision>
+            <density>4000</density>
             <origin xyz="0 0.0 0.0" rpy="0 0.0 0" />
             <geometry>
@@ -286,9 +355,6 @@
                 <friction>
                     <ode>
-                        <mu>1.0</mu>
-                        <mu2>100</mu2>
-                        <fdir1>0 0 0</fdir1>
-                        <slip1>0.02</slip1>
-                        <slip2>0</slip2>
+                        <mu>10000000</mu>
+                        <mu2>10000000</mu2>
                     </ode>
                 </friction>
@@ -298,11 +364,16 @@
     <!-- 右前轮 -->
     <link name="right_wheel_link">
-        <inertial>
+        <!-- <inertial>
+            <origin xyz="0 0.0 0.0" rpy="-1.5707 0.0 -1.5707" />
+            <mass value="30.0" />
+            <inertia ixx="0.089" ixy="0.0" ixz="0.0" iyy="0.089" iyz="0.0" izz="0.172" />
+        </inertial> -->
+        <inertial auto="true">
+            <origin xyz="0 0.0 0.0" rpy="-1.5707 0.0 -1.5707" />
+            <mass value="5.0" />
+            <inertia ixx="0.089" ixy="0.0" ixz="0.0" iyy="0.089" iyz="0.0" izz="0.172" />
+        </inertial>
+        <visual>
             <origin xyz="0 0.0 0.0" rpy="0 0.0 0" />
-            <mass value="30.0" />
-            <inertia ixx="10" ixy="0.0" ixz="0.0" iyy="12" iyz="0.0" izz="12" />
-        </inertial>
-        <visual>
-            <origin xyz="0 0.0 0.0" rpy="0 0.0 0" />
             <geometry>
                 <mesh filename="package://car_description/meshes/frontwheel.stl" scale="0.0010 0.0010 0.0010" />
@@ -311,4 +382,5 @@
         </visual>
         <collision>
+            <density>4000</density>
             <origin xyz="0 0.0 0.0" rpy="0 0.0 0" />
             <geometry>
@@ -318,9 +390,6 @@
                 <friction>
                     <ode>
-                        <mu>1.0</mu>
-                        <mu2>100</mu2>
-                        <fdir1>0 0 0</fdir1>
-                        <slip1>0.02</slip1>
-                        <slip2>0</slip2>
+                        <mu>10000000</mu>
+                        <mu2>10000000</mu2>
                     </ode>
                 </friction>
@@ -333,5 +402,5 @@
             <origin xyz="0.0 0.0 0.0" rpy="0.0 0.0 0.0" />
             <mass value="3.0" />
-            <inertia ixx="0.054" ixy="0.0" ixz="0.0" iyy="0.252" iyz="0.0" izz="0.252" />
+            <inertia ixx="0.0158" ixy="0.0" ixz="0.0" iyy="0.0158" iyz="0.0" izz="0.005" />
         </inertial>
     </link>
@@ -402,14 +471,14 @@
         <child link="fork"/>
         <axis xyz="0.0 0.0 1"/>
-        <limit lower="-1" upper="3.0" effort="3000.0" velocity="1.0"/>
-        <dynamics damping="100.0" friction="10"/>
+        <limit lower="-0.1" upper="3.0" effort="3000.0" velocity="1.0"/>
+        <dynamics damping="10.0" friction="50.0"/>
     </joint>
     <joint name="main_wheel_base_joint" type="continuous">
-        <origin xyz="0.21 0.0 0.04" rpy="0.0 0.0 0.0"/>
+        <origin xyz="0.25 0.0 0.05" rpy="0.0 0.0 0.0"/>
         <parent link="footbase"/>
         <child link="main_wheel_base_link"/>
         <axis xyz="0.0 0.0 1"/>
-        <limit effort="500.0" velocity="1"/>
-        <dynamics damping="1.0" friction="1"/>
+        <limit effort="500.0" velocity="2"/>
+        <dynamics damping="1.0" friction="30"/>
     </joint>
     <joint name="main_wheel_joint" type="continuous">
@@ -418,6 +487,6 @@
         <child link="main_wheel_link"/>
         <axis xyz="0.0 1.0 0.0"/>
-        <limit effort="1600.0" velocity="20.0"/>
-        <dynamics damping="4.0" friction="10.0" friction2="100.0"/>
+        <limit effort="700.0" velocity="200.0"/>
+        <dynamics damping="0.1" friction="1.0"/>
     </joint>
     <joint name="left_wheel_joint" type="continuous">
@@ -426,6 +495,6 @@
         <child link="left_wheel_link"/>
         <axis xyz="1.0 0.0 0.0"/>
-        <limit lower="-100" upper="100.0" effort="20.0" velocity="2.0"/>
-        <dynamics damping="1.0" friction="10.0" friction2="100.0"/>
+        <limit effort="200.0" velocity="200.0"/>
+        <dynamics damping="0.1" friction="1.0" />
     </joint>
     <joint name="right_wheel_joint" type="continuous">
@@ -434,6 +503,6 @@
         <child link="right_wheel_link"/>
         <axis xyz="1.0 0.0 0.0"/>
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
Commit message: 反光率设置

File: src/car_description/urdf/buggy3.urdf.xacro (robot description, xacro)
@@ -466,4 +466,10 @@
         <child link="sun"/>
     </joint>
+    <joint name="base_link_joint" type="fixed">
+        <origin xyz="1.01 0 0" rpy="0.0 0.0 0"/>
+        <parent link="base_link"/>
+        <child link="footbase"/>
+        <axis xyz="0.0 0.0 0.0"/>
+    </joint>
     <joint name="fork_joint" type="prismatic">
         <origin xyz="0.0 0.0 0.0" rpy="0.0 0.0 0.0"/>
@@ -471,5 +477,5 @@
         <child link="fork"/>
         <axis xyz="0.0 0.0 1"/>
-        <limit lower="-0.1" upper="3.0" effort="3000.0" velocity="1.0"/>
+        <limit lower="0" upper="3.0" effort="3000.0" velocity="1.0"/>
         <dynamics damping="10.0" friction="50.0"/>
     </joint>
@@ -479,5 +485,5 @@
         <child link="main_wheel_base_link"/>
         <axis xyz="0.0 0.0 1"/>
-        <limit effort="500.0" velocity="2"/>
+        <limit effort="500.0" velocity="0.3"/>
         <dynamics damping="1.0" friction="30"/>
     </joint>
@@ -506,10 +512,4 @@
         <dynamics damping="0.1" friction="1.0"/>
     </joint>
-    <joint name="base_link_joint" type="fixed">
-        <origin xyz="-1.01 0 0" rpy="0.0 0.0 0"/>
-        <parent link="footbase"/>
-        <child link="base_link"/>
-        <axis xyz="0.0 0.0 0.0"/>
-    </joint>
     <!-- ros2_control -->
     <ros2_control name="GazeboSimSystem" type="system">
@@ -518,7 +518,7 @@
         </hardware>
         <joint name="fork_joint">
-            <command_interface name="position">
-                <param name="min">0</param>
-                <param name="max">3</param>
+            <command_interface name="velocity">
+                <param name="min">-10</param>
+                <param name="max">10</param>
             </command_interface>
             <state_interface name="position" />
@@ -572,12 +572,12 @@
                 <scan>
                     <horizontal>
-                        <samples>3600</samples>
+                        <samples>16000</samples>
                         <resolution>1</resolution>
-                        <min_angle>-2.35619</min_angle>
-                        <max_angle>2.35619</max_angle>
+                        <min_angle>-3.14159</min_angle>
+                        <max_angle>3.14159</max_angle>
                     </horizontal>
                     <vertical>
                         <samples>1</samples>
-                        <resolution>0.01</resolution>
+                        <resolution>1</resolution>
                         <min_angle>0</min_angle>
                         <max_angle>0</max_angle>
@@ -604,5 +604,5 @@
         <sensor name="imu" type="imu">
             <always_on>true</always_on>
-            <update_rate>1000</update_rate>
+            <update_rate>200</update_rate>
             <visualize>true</visualize>
             <topic>imu</topic>

Commit message: 里程记辅助的匹配

File: src/car_description/urdf/buggy3.urdf.xacro (robot description, xacro)
@@ -421,9 +421,4 @@
         </inertial>
     </link>
-    <joint name="main_2d_lidar_foot_joint" type="fixed">
-        <origin xyz="0.115 0.0 1.9" rpy="0.0 0.0 0.0"/>
-        <parent link="footbase"/>
-        <child link="main_2d_lidar_link"/>
-    </joint>
     <joint name="frame_foot_joint" type="fixed">
         <origin xyz="0.0 0.0 0.0" rpy="0.0 0.0 0.0"/>
@@ -467,8 +462,13 @@
     </joint>
     <joint name="base_link_joint" type="fixed">
-        <origin xyz="1.01 0 0" rpy="0.0 0.0 0"/>
-        <parent link="base_link"/>
+        <origin xyz="-1.01 0 0" rpy="0.0 0.0 0"/>
+        <parent link="footbase"/>
+        <child link="base_link"/>
+        <axis xyz="0.0 0.0 0.0"/>
+    </joint>
+    <joint name="foot_main_2d_lidar_joint" type="fixed">
+        <origin xyz="-0.115 0.0 -1.9" rpy="0.0 0.0 0.0"/>
+        <parent link="main_2d_lidar_link"/>
         <child link="footbase"/>
-        <axis xyz="0.0 0.0 0.0"/>
     </joint>
     <joint name="fork_joint" type="prismatic">
